Commit message: test for grasp

File: panda_sim_description/urdf/panda_sim_description.urdf.xacro (robot description, xacro)
@@ -35,16 +35,23 @@
     <xacro:hand ns="panda" rpy="0 0 0" connected_to="panda_link8"/>
     <!-- bottle1 -->
-    <xacro:include filename="$(find panda_sim_description)/urdf/bottle1.urdf.xacro" />
+    <!--xacro:include filename="$(find panda_sim_description)/urdf/bottle1.urdf.xacro" /-->
     <!-- bottle2 -->
-    <xacro:include filename="$(find panda_sim_description)/urdf/bottle2.urdf.xacro" />
-    <joint name="table_to_bottle1" type="fixed">
+    <!--xacro:include filename="$(find panda_sim_description)/urdf/bottle2.urdf.xacro" /-->
+    <!--joint name="table_to_bottle1" type="fixed">
              <origin xyz="0.2 0.04 0.04" rpy="0 0 0" />
              <parent link="tabletop_ontop"/>
              <child link="bottle1_link"/>
-    </joint>
-    <joint name="table_to_bottle2" type="fixed">
+    </joint-->
+    <!--joint name="table_to_bottle2" type="fixed">
              <origin xyz="0.2 -0.04 0.04" rpy="0 0 0" />
              <parent link="tabletop_ontop"/>
              <child link="bottle2_link"/>
+    </joint-->
+    <!-- box -->
+    <xacro:include filename="$(find panda_sim_gazebo)/objects/basic_cube.urdf" />
+    <joint name="table_to_basic_box" type="fixed">
+             <origin xyz="0.2 0.04 0.04" rpy="0 0 0" />
+             <parent link="tabletop_ontop"/>
+             <child link="cube_link"/>
     </joint>
     <!--

File: panda_sim_gazebo/objects/basic_cube.urdf (robot description, URDF)
Before this commit: robot basic_box, 1 links, 0 joints
Links:
- removed link box_link
- added link cube_link, mass 0.01; collision box size=0.2 0.04 0.04; visual box size=0.2 0.04 0.04
