Commit message: added grasp

File: panda_sim_description/urdf/hand.xacro (robot description, xacro)
@@ -21,15 +21,12 @@
       </collision>
       <inertial>
-        <origin xyz="-0.000025 0.005735 0.103826" rpy="0 0 0"/>
-          <mass value="0.73"/>
-          <inertia
-            ixx="0.001405" ixy="0.0"    ixz="0.0"
-                        iyy="0.000202" iyz="0.0"
-                                     izz="0.001293"/>
+        <mass value="0.73" />
+        <origin xyz="0 0.0015244 0.0275912" rpy="0 0 0" />
+        <inertia ixx="0.00278560230025" ixy="0.0" ixz="0.0" iyy="0.000400033405336" iyz="0.0" izz="0.00256378041832" />
       </inertial>
     </link>
   <gazebo reference="${ns}_hand">
-      <mu1>100.0</mu1>
-      <mu2>100.0</mu2>
+      <mu1>0.61</mu1>
+      <mu2>0.61</mu2>
     </gazebo>
     <link name="${ns}_leftfinger">
@@ -45,15 +42,12 @@
       </collision>
       <inertial>
-        <origin xyz="0.000002  0.014564 0.022794" rpy="0 0 0"/>
-          <mass value="1.1e-3"/>
-          <inertia
-            ixx="0.00000338" ixy="0"          ixz="0"
-                             iyy="0.00000332" iyz="0.0000006"
-                                              izz="0.00000078"/>
+        <mass value="0.1" />
+        <origin xyz="0 0.0145644 0.0227941" rpy="0 0 0" />
+        <inertia ixx="3.01220925051e-05" ixy="0.0" ixz="0.0" iyy="2.95873808038e-05" iyz="0.0" izz="6.95125211657e-06" />
       </inertial>
     </link>
     <gazebo reference="${ns}_leftfinger">
-      <mu1>100.0</mu1>
-      <mu2>100.0</mu2>
+      <mu1>0.61</mu1>
+      <mu2>0.61</mu2>
     </gazebo>
     <link name="${ns}_rightfinger">
@@ -70,16 +64,13 @@
         </geometry>
       </collision>
-      <inertial>
-        <origin xyz="0.000002  0.014564 0.022794" rpy="0 0 ${pi}"/>
-          <mass value="1.1e-3"/>
-          <inertia
-            ixx="0.00000338" ixy="0"          ixz="0"
-                             iyy="0.00000332" iyz="0.0000006"
-                                              izz="0.00000078"/>
+       <inertial>
+        <mass value="0.1" />
+        <origin xyz="0 0.0145644 0.0227941" rpy="0 0 ${pi}" />
+        <inertia ixx="3.01220925051e-05" ixy="0.0" ixz="0.0" iyy="2.95873808038e-05" iyz="0.0" izz="6.95125211657e-06" />
       </inertial>
     </link>
     <gazebo reference="${ns}_rightfinger">
-      <mu1>100.0</mu1>
-      <mu2>100.0</mu2>
+      <mu1>0.61</mu1>
+      <mu2>0.61</mu2>
     </gazebo>
     <joint name="${ns}_finger_joint1" type="prismatic">
