Commit message: Trying different objects

File: panda_sim_gazebo/objects/basic_cylinder.urdf (robot description, URDF)
Before this commit: robot basic_cylinder, 1 links, 0 joints
Links:
- link cylinder_link: geometry collision cylinder length=0.15 radius=0.02; visual cylinder length=0.15 radius=0.02

File: panda_sim_gazebo/objects/basic_sphere.urdf (robot description, URDF)
Before this commit: robot basic_sphere, 1 links, 0 joints
Links:
- link sphere_link: geometry collision sphere radius=0.02; visual sphere radius=0.02

Commit message: implemented the complex model

File: panda_sim_gazebo/objects/basic_cylinder.urdf (robot description, URDF)
Before this commit: robot basic_cylinder, 1 links, 0 joints
Links:
- link cylinder_link: geometry collision cylinder length=0.15 radius=0.03; visual cylinder length=0.15 radius=0.03
